File: breadboard_psu.kicad_pcb (KiCad board)
At the start: 2 copper layers, 58.4 x 71.1 mm, 22 parts, among them J1 Barrel_Jack_MountingPin, J2 Conn_02x02_Odd_Even, J3 Conn_02x02_Odd_Even, J4 Conn_02x04_Odd_Even, J5 Conn_01x02, SW1 SW_DPDT_x2, SW2 SW_DPDT_x2, U1 LM317_TO-220

Commit message: Ajout JLCJLCJLCJLC silkscreen bottom
Other:
- board text added: "JLCJLCJLCJLC"
Changed lines of the file:
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@@
       (drillshape 0)
       (scaleselection 1)
-      (outputdirectory "documentation")
+      (outputdirectory "gerber")
     )
   )
@@
   (gr_arc locked (start 137.0584 77.978) (mid 137.430374 77.079974) (end 138.3284 76.708)
     (stroke (width 0.2) (type default)) (layer "Edge.Cuts"))
+  (gr_text "JLCJLCJLCJLC" (at 114.7064 130.048) (layer "B.SilkS")
+    (effects (font (size 0.762 0.762) (thickness 0.1524) bold) (justify bottom mirror))
+  )
   (gr_text "PCB rev. 1" (at 93.3704 121.92 90) (layer "B.SilkS")
     (effects (font (size 1.5 1.5) (thickness 0.3) bold) (justify right mirror))
@@
     (height 40.132)
     (orientation 1)
-    (gr_text "2800,0000 mils" (at 174.768 95.25 90) (layer "F.Fab")
+    (gr_text "2800.0000 mils" (at 174.768 95.25 90) (layer "F.Fab")
       (effects (font (size 1 1) (thickness 0.1524)))
     )
@@
     (height 34.036)
     (orientation 1)
-    (gr_text "2500,0000 mils" (at 165.632 95.25 90) (layer "F.Fab")
+    (gr_text "2500.0000 mils" (at 165.632 95.25 90) (layer "F.Fab")
       (effects (font (size 1.5 1.5) (thickness 0.1524)))
     )
@@
     (height -11.43)
     (orientation 0)
-    (gr_text "1470,0000 mils" (at 114.5794 50.9176) (layer "F.Fab")
+    (gr_text "1470.0000 mils" (at 114.5794 50.9176) (layer "F.Fab")
       (effects (font (size 1 1) (thickness 0.1524)))
     )
@@
     (height 9.906)
     (orientation 1)
-    (gr_text "1860,0000 mils" (at 156.234 95.25 90) (layer "F.Fab")
+    (gr_text "1860.0000 mils" (at 156.234 95.25 90) (layer "F.Fab")
       (effects (font (size 1.5 1.5) (thickness 0.1524)))
     )
@@
     (height -13.97)
     (orientation 0)
-    (gr_text "1770,0000 mils" (at 114.5794 45.8376) (layer "F.Fab")
+    (gr_text "1770.0000 mils" (at 114.5794 45.8376) (layer "F.Fab")
       (effects (font (size 1 1) (thickness 0.1524)))
     )
